Commit message: 更新简易运动学仿真

File: resources/arm.urdf.xacro (robot description, xacro)
@@ -1,25 +1,21 @@
 <?xml version="1.0"?>
-<robot name="left_arm">
+<robot name="right_arm">
   <link name="base_link"/>
-  <link name="link1"/>
-  <link name="link2"/>
-  <link name="link3"/>
-  <link name="link4"/>
-  <link name="link5"/>
-  <link name="link6"/>
   <joint name="j1" type="revolute">
     <parent link="base_link"/>
     <child link="link1"/>
-    <origin xyz="0.26 0 0" rpy="0 0 0"/>
+    <origin xyz="0.04 0 0" rpy="0 0 0"/>
     <axis xyz="0 0 1"/>
     <limit lower="-2.9670597" upper="2.9670597" effort="100" velocity="2"/>
   </joint>
+  <link name="link1"/>
   <joint name="j2" type="revolute">
     <parent link="link1"/>
     <child link="link2"/>
     <origin xyz="0.24 0 0" rpy="0 0 0"/>
-    <axis xyz="0 1 0"/>
+    <axis xyz="1 0 0"/>
     <limit lower="-2.0943951" upper="2.0943951" effort="100" velocity="2"/>
   </joint>
+  <link name="link2"/>
   <joint name="j3" type="revolute">
     <parent link="link2"/>
@@ -29,4 +25,5 @@
     <limit lower="-2.9670597" upper="2.9670597" effort="100" velocity="2"/>
   </joint>
+  <link name="link3"/>
   <joint name="j4" type="revolute">
     <parent link="link3"/>
@@ -36,4 +33,5 @@
     <limit lower="-3.2288591" upper="3.2288591" effort="100" velocity="2"/>
   </joint>
+  <link name="link4"/>
   <joint name="j5" type="revolute">
     <parent link="link4"/>
@@ -43,10 +41,12 @@
     <limit lower="-2.0943951" upper="2.0943951" effort="100" velocity="2"/>
   </joint>
+  <link name="link5"/>
   <joint name="j6" type="revolute">
     <parent link="link5"/>
     <child link="link6"/>
-    <origin xyz="0.06 0 0" rpy="0 0 0"/>
-    <axis xyz="1 0 0"/>
+    <origin xyz="0.1 0 0" rpy="0 0 0"/>
+    <axis xyz="0 0 1"/>
     <limit lower="-6.2831853" upper="6.2831853" effort="100" velocity="2"/>
   </joint>
+  <link name="link6"/>
 </robot>
